File: hardware/uMidi.sch (KiCad schematic (older format))
At the start: 61 parts, among them CON1 USB-MINI-B, IC1 ATXMEGA128A4U-M, IC2 74LS14, IC3 LT1129CST-3.3, IC4 6N138, P1 MIDI Out, P2 MIDI Out, P3 MIDI Out, P4 MIDI Out, P5 MIDI Out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

Commit message: Add and use led 0603 footprint
Parts:
- D7, D8: footprint (none) -> uMIDI:LED-0603
Changed lines of the file:
@@
 F 0 "D7" H 6350 3400 50  0000 C CNN
 F 1 "LED Green" H 6350 3200 50  0000 C CNN
-F 2 "" H 6350 3300 60  0001 C CNN
+F 2 "uMIDI:LED-0603" H 6350 3300 60  0001 C CNN
 F 3 "http://optoelectronics.liteon.com/upload/download/DS22-2000-228/S_110_LTST-C191KGKT.pdf" H 6350 3300 60  0001 C CNN
 F 4 "LTST-C191KGKT" H 6350 3400 50  0001 C CNN "Manufacturer Part Number"
@@
 F 0 "D8" H 6350 3700 50  0000 C CNN
 F 1 "LED Red" H 6350 3500 50  0000 C CNN
-F 2 "" H 6350 3600 60  0001 C CNN
+F 2 "uMIDI:LED-0603" H 6350 3600 60  0001 C CNN
 F 3 "http://optoelectronics.liteon.com/upload/download/DS22-2000-223/S_110_LTST-C191KRKT.pdf" H 6350 3600 60  0001 C CNN
 F 4 "LTST-C191KRKT" H 6350 3700 50  0001 C CNN "Manufacturer Part Number"
