File: hardware/uMidi.sch (KiCad schematic (older format))
At the start: 61 parts, among them CON1 USB-MINI-B, IC1 ATXMEGA128A4U-M, IC2 74LS14, IC3 LT1129CST-3.3, IC4 6N138, P1 MIDI In, P2 MIDI Thru, P3 MIDI T/O, P4 MIDI Out, P5 5..12 V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

Commit message: Swap red and green LEDs according to doc
Parts:
- D7: value LED Green -> LED Red; Manufacturer Part Number LTST-C191KGKT -> LTST-C191KRKT; Supplier Link https://www.digikey.de/product-detail/de/LTST-C191KGKT/160-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 -> https://www.digikey.de/product-detail/de/LTST-C191KRKT/160-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; Supplier Part Number 160-1446-1-ND -> 160-1447-1-ND
- D8: value LED Red -> LED Green; Manufacturer Part Number LTST-C191KRKT -> LTST-C191KGKT; Supplier Link https://www.digikey.de/product-detail/de/LTST-C191KRKT/160-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 -> https://www.digikey.de/product-detail/de/LTST-C191KGKT/160-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; Supplier Part Number 160-1447-1-ND -> 160-1446-1-ND
Changed lines of the file:
@@
 P 6350 3300
 F 0 "D7" H 6350 3400 50  0000 C CNN
-F 1 "LED Green" H 6350 3200 50  0000 C CNN
+F 1 "LED Red" H 6350 3200 50  0000 C CNN
 F 2 "" H 6350 3300 60  0001 C CNN
-F 3 "http://optoelectronics.liteon.com/upload/download/DS22-2000-228/S_110_LTST-C191KGKT.pdf" H 6350 3300 60  0001 C CNN
-F 4 "LTST-C191KGKT" H 6350 3400 50  0001 C CNN "Manufacturer Part Number"
+F 3 "http://optoelectronics.liteon.com/upload/download/DS22-2000-223/S_110_LTST-C191KRKT.pdf" H 6350 3300 60  0001 C CNN
+F 4 "LTST-C191KRKT" H 6350 3400 50  0001 C CNN "Manufacturer Part Number"
 F 5 "Digikey" H 6350 3400 50  0001 C CNN "Supplier"
-F 6 "https://www.digikey.de/product-detail/de/LTST-C191KGKT/160-1446-1-ND/386834" H 6350 3400 50  0001 C CNN "Supplier Link"
+F 6 "https://www.digikey.de/product-detail/de/LTST-C191KRKT/160-1447-1-ND/386836" H 6350 3400 50  0001 C CNN "Supplier Link"
 F 7 "Lite-On Inc." H 6350 3400 50  0001 C CNN "Manufacturer"
-F 8 "160-1446-1-ND" H 6350 3400 50  0001 C CNN "Supplier Part Number"
+F 8 "160-1447-1-ND" H 6350 3400 50  0001 C CNN "Supplier Part Number"
 	1    6350 3300
 	-1   0    0    1
@@
 P 6350 3600
 F 0 "D8" H 6350 3700 50  0000 C CNN
-F 1 "LED Red" H 6350 3500 50  0000 C CNN
+F 1 "LED Green" H 6350 3500 50  0000 C CNN
 F 2 "" H 6350 3600 60  0001 C CNN
-F 3 "http://optoelectronics.liteon.com/upload/download/DS22-2000-223/S_110_LTST-C191KRKT.pdf" H 6350 3600 60  0001 C CNN
-F 4 "LTST-C191KRKT" H 6350 3700 50  0001 C CNN "Manufacturer Part Number"
-F 5 "160-1447-1-ND" H 6350 3700 50  0001 C CNN "Supplier Part Number"
-F 6 "https://www.digikey.de/product-detail/de/LTST-C191KRKT/160-1447-1-ND/386836" H 6350 3700 50  0001 C CNN "Supplier Link"
+F 3 "http://optoelectronics.liteon.com/upload/download/DS22-2000-228/S_110_LTST-C191KGKT.pdf" H 6350 3600 60  0001 C CNN
+F 4 "LTST-C191KGKT" H 6350 3700 50  0001 C CNN "Manufacturer Part Number"
+F 5 "160-1446-1-ND" H 6350 3700 50  0001 C CNN "Supplier Part Number"
+F 6 "https://www.digikey.de/product-detail/de/LTST-C191KGKT/160-1446-1-ND/386834" H 6350 3700 50  0001 C CNN "Supplier Link"
 F 7 "Lite-On Inc." H 6350 3700 50  0001 C CNN "Manufacturer"
 F 8 "Digikey" H 6350 3700 50  0001 C CNN "Supplier"
